File: PCB/RVSP_Pocket/RVSP_Pocket.kicad_pcb (KiCad board)
At the start: 4 copper layers, 87.7 x 37.6 mm, 72 parts, among them Q1 8205A_C5148694, SW1 SW_Push, U1 STM32F401CCUx, U2 AMS1117-3.3, U3 MT3608, U4 TP4056-42-ESOP8, U5 DW01A, U6 TPS2116DRL, Y1 25 Mhz

Commit message: Added readme
Parts:
- added G***: LOGO, LOGO, B.Cu at (102.2, 74.4)
- moved G*** 70.8 mm to (164.4, 81.5)
- moved G*** 70.4 mm to (164.2, 75.2)
Other:
- board text added: ">> How fast can you read? <<"
- board text added: "V1.0"
