File: PCB/RVSP_Pocket/power.kicad_sch (KiCad schematic)
At the start: 0 parts

Commit message: Added PCB files
Parts:
- added BatteryPort1: Conn_01x02, TestPoint:TestPoint_2Pads_Pitch5.08mm_Drill1.3mm, symbol Connector_Generic:Conn_01x02
- added C13, C14: 22u, Capacitor_SMD:C_0603_1608Metric_Pad1.08x0.95mm_HandSolder, symbol Device:C
- added C17, C18: 22uF, Capacitor_SMD:C_0603_1608Metric_Pad1.08x0.95mm_HandSolder, symbol Device:C
- added C19: 100n, Capacitor_SMD:C_0603_1608Metric_Pad1.08x0.95mm_HandSolder, symbol Device:C
- added C20: 10u, Capacitor_SMD:C_0603_1608Metric_Pad1.08x0.95mm_HandSolder, symbol Device:C
- added D1, D4: GREEN, LED_SMD:LED_0805_2012Metric_Pad1.15x1.40mm_HandSolder, symbol Device:LED
- added D2: SS34, Diode_SMD:D_SMA, symbol Diode:SS34
- added D3: BLUE, LED_SMD:LED_0805_2012Metric_Pad1.15x1.40mm_HandSolder, symbol Device:LED
- added DOWN, RIGHT, SELECT, UP: SW_Push, LK_lib:SW_PUSH_6mm_H5mm_2Leg, symbol Switch:SW_Push
- added H1, H2, H3, H4: MountingHole, MountingHole:MountingHole_3.2mm_M3_DIN965, symbol Mechanical:MountingHole
- added L1: 22uH, Inductor_SMD:L_10.4x10.4_H4.8, symbol Device:L
- added Q1: 8205A_C5148694, EasyEDA:TSSOP-8_L4.4-W3.0-P0.65-LS6.4-BL, symbol EasyEDA:8205A_C5148694
- added R1, R2: 5.1k, Resistor_SMD:R_0603_1608Metric_Pad0.98x0.95mm_HandSolder, symbol Device:R
- added R10, R11, R14, R3: 1k, Resistor_SMD:R_0603_1608Metric_Pad0.98x0.95mm_HandSolder, symbol Device:R
- added R12: 470, Resistor_SMD:R_0603_1608Metric_Pad0.98x0.95mm_HandSolder, symbol Device:R
- added R13: 2k, Resistor_SMD:R_0603_1608Metric_Pad0.98x0.95mm_HandSolder, symbol Device:R
- added R15, R16: 470k, Resistor_SMD:R_0603_1608Metric_Pad0.98x0.95mm_HandSolder, symbol Device:R
- added R17: 150, Resistor_SMD:R_0603_1608Metric_Pad0.98x0.95mm_HandSolder, symbol Device:R
- added R18: 10k, Resistor_SMD:R_0603_1608Metric_Pad0.98x0.95mm_HandSolder, symbol Device:R
- added R19, R20: 47k, Resistor_SMD:R_0603_1608Metric_Pad0.98x0.95mm_HandSolder, symbol Device:R
- added R8: 390k, Resistor_SMD:R_0603_1608Metric_Pad0.98x0.95mm_HandSolder, symbol Device:R
- added R9: 51K, Resistor_SMD:R_0603_1608Metric_Pad0.98x0.95mm_HandSolder, symbol Device:R
- added TP1, TP2: TestPoint, TestPoint:TestPoint_Pad_D2.0mm, symbol Connector:TestPoint
- added U2: AMS1117-3.3, Package_TO_SOT_SMD:SOT-223-3_TabPin2, symbol Regulator_Linear:AMS1117-3.3
- added U3: MT3608, Package_TO_SOT_SMD:SOT-23-6, symbol Regulator_Switching:MT3608
- added U4: TP4056-42-ESOP8, Package_SO:SOIC-8-1EP_3.9x4.9mm_P1.27mm_EP2.41x3.3mm_ThermalVias, symbol Battery_Management:TP4056-42-ESOP8
- added U5: DW01A, Package_TO_SOT_SMD:SOT-23-6, symbol Battery_Management:DW01A
- added U6: TPS2116DRL, Package_TO_SOT_SMD:SOT-583-8, symbol Power_Management:TPS2116DRL
- added USB_C1: USB_C_Receptacle_USB2.0_16P, Connector_USB:USB_C_Receptacle_GCT_USB4105-xx-A_16P_TopMnt_Horizontal, symbol Connector:USB_C_Receptacle_USB2.0_16P
Connections:
- new net: R13.2, U5.2 (CS)
- new net: C19.1, R12.2, U5.5 (VCC)
- new net: R8.2, R9.1, U3.3 (FB)
- new net: R1.2, USB_C1.A5 (CC1)
- new net: D3.1 (K), R10.1
- new net: D2.2 (A), L1.2, TP2.1, U3.1 (SW)
- new net: D4.1 (K), R11.1
- new net: D1.1 (K), R3.1
- new net: R2.2, USB_C1.B5 (CC2)
- new net: R14.2, R17.1
- new net +3V3: C13.1, D1.2 (A), U2.2 (VO)
- new net BAT_5V: C18.1, D2.1 (K), R8.1, U6.6 (VIN2)
- new net BAT_LVL: R15.2, R16.1
- new net BAT_Neg: BatteryPort1.2 (Pin_2), C19.2, Q1.7 (S2), U5.6 (GND)
- new net BAT_ON: R18.1, U6.8 (ST)
- new net BAT_Pos: BatteryPort1.1 (Pin_1), C17.1, L1.1, R12.1, R15.1, TP1.1, U3.4 (EN), U3.5 (IN), U4.5 (BAT)
- new net D1: Q1.1 (D1), Q1.8 (D2)
- new net DWN_BTN: DOWN.1
- new net GND: C13.2, C14.2, C17.2, C18.2, C20.2, DOWN.2, Q1.2 (S1), R1.1, R13.1, R16.2, R17.2, R2.1, R20.2, R3.2, R9.2, RIGHT.2, SELECT.2, U2.1 (GND), U3.2 (GND), U4.1 (TEMP), U4.3 (GND), U4.9 (EPAD), U6.1 (GND), UP.2, USB_C1.A1 (GND), USB_C1.A12 (GND), USB_C1.B1 (GND), USB_C1.B12 (GND)
- new net OC: Q1.5 (G2), U5.3 (OC)
- new net OD: Q1.4 (G1), U5.1 (OD)
- new net PR1: R19.2, R20.1, U6.4 (PR1)
- new net PROG: R14.1, U4.2 (PROG)
- new net REG_IN: C14.1, U2.3 (VI), U6.2 (VOUT), U6.7 (VOUT)
- new net RIGHT_BTN: RIGHT.1
- new net SELECT_BTN: SELECT.1
- new net UP_BTN: UP.1
- new net USB_D+: USB_C1.A6 (D+), USB_C1.B6 (D+)
- new net USB_D-: USB_C1.A7 (D-), USB_C1.B7 (D-)
- new net VBUS: C20.1, D3.2 (A), D4.2 (A), R18.2, R19.1, U4.4 (V_{CC}), U4.8 (CE), U6.3 (VIN1), U6.5 (MODE), USB_C1.A4 (VBUS), USB_C1.A9 (VBUS), USB_C1.B4 (VBUS), USB_C1.B9 (VBUS)
- new net ~{CHRG}: R10.2, U4.7 (~{CHRG})
- new net ~{STDBY}: R11.2, U4.6 (~{STDBY})
- no-connect marks 0 -> 5
Other:
- note added: "*Internal pull-up resistors"
- note added: "3.3V Regulator"
- note added: "BAT_LVL = BAT_POS/2 BAT_POS_MAX = 4.2V so any GPIO is ok"
- note added: "Boost Convertor"
- note added: "IBAT = 1/(RISET) * 1200 18650 has 2600mAh with CC = 0.5C -> IBAT_MAX = 1300 mA"
- note added: "No TEMP monitoring due to low risk Future versions could include a 10 kOhm NTC for extra protection"
- note added: "Note: The input voltage of REG_IN must be >= 1.2V than input Otherwise the regulator cannot reliably produce 3.3V output See regulator drop-out voltage"
- note added: "Power Mux + Monitoring"
- note added: "TP4056 Charging + Protection Circuit"
- note added: "USB_C 16P"

Commit message: Added readme
Parts:
- renumbered DOWN to DOWN1, RIGHT to RIGHT1, SELECT to SELECT1, UP to UP1
Changed lines of the file:
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@@
 		(dnp no)
 		(fields_autoplaced yes)
-		(property "Reference" "DOWN"
+		(property "Reference" "DOWN1"
 			(at 40.64 113.03 0)
 			(show_name no)
@@
 			(project "RVSP_Pocket"
 				(path "/68d24f2b-0e73-4817-9bb9-fc791efd9ec9"
-					(reference "DOWN")
+					(reference "DOWN1")
 					(unit 1)
 				)
@@
 		(dnp no)
 		(fields_autoplaced yes)
-		(property "Reference" "UP"
+		(property "Reference" "UP1"
 			(at 40.64 124.46 0)
 			(show_name no)
@@
 			(project "RVSP_Pocket"
 				(path "/68d24f2b-0e73-4817-9bb9-fc791efd9ec9"
-					(reference "UP")
+					(reference "UP1")
 					(unit 1)
 				)
@@
 		(dnp no)
 		(fields_autoplaced yes)
-		(property "Reference" "SELECT"
+		(property "Reference" "SELECT1"
 			(at 40.64 137.16 0)
 			(show_name no)
@@
 			(project "RVSP_Pocket"
 				(path "/68d24f2b-0e73-4817-9bb9-fc791efd9ec9"
-					(reference "SELECT")
+					(reference "SELECT1")
 					(unit 1)
 				)
@@
 		(dnp no)
 		(fields_autoplaced yes)
-		(property "Reference" "RIGHT"
+		(property "Reference" "RIGHT1"
 			(at 40.64 101.6 0)
 			(show_name no)
@@
 			(project "RVSP_Pocket"
 				(path "/68d24f2b-0e73-4817-9bb9-fc791efd9ec9"
-					(reference "RIGHT")
+					(reference "RIGHT1")
 					(unit 1)
 				)
